File: Coffee_Machine_Gogokhia_Edition_SIMPLE_V1.0/PCB/Boiler.kicad_sch (KiCad schematic)
At the start: 16 parts

Commit message: Edited
Parts:
- removed C? (x2): .01uF, Capacitor_THT:C_Disc_D5.0mm_W2.5mm_P5.00mm, symbol Device:C
- removed J?: BOILER_TAB_Cap, MyLibrary:TAB_CONN, symbol Connector:Conn_01x01_Male
- removed Q?: BTA16, Package_TO_SOT_THT:TO-220-3_Vertical, symbol Triac_Thyristor:BTA16-600B
- removed R?: 330R, Resistor_SMD:R_0603_1608Metric, symbol Device:R
- removed R? (x2): 39R, Resistor_SMD:R_1206_3216Metric, symbol Device:R
- removed R?: 10K, Resistor_SMD:R_0603_1608Metric, symbol Device:R
- removed R?: 180R, Resistor_SMD:R_1206_3216Metric, symbol Device:R
- removed U?: MOC3021M, MyLibrary:OPTOCOUPLER_H11F3SR2M, symbol Relay_SolidState:MOC3021M
- J9: renamed from J?; footprint MyLibrary:TAB_CONN -> Footprint:TAB_Conn
- Q3: renamed from Q?; footprint Package_TO_SOT_THT:TO-220-3_Vertical -> Footprint:BTA16_wH_SINK
- U6: renamed from U?; footprint MyLibrary:OPTOCOUPLER_H11F3SR2M -> Footprint:DIP6_SMD
- gave numbers to parts that had none: 3
Other:
- note removed: "BOILER_Cap"
