File: Coffee_Machine_Gogokhia_Edition_SIMPLE_V1.0/PCB/Coffe_Machine_Gogokhia_Edition_SIMPLE.kicad_pcb (KiCad board)
At the start: 2 copper layers, 150 x 100 mm, 181 parts, among them J1 NEUT_TAB, J10 Conn_01x02, J11 SW, J12 SW3_TAB, J13 Conn_01x02, J14 SW1_TAB, J15 SW2_TAB, J16 Conn_01x02, J17 Conn_01x02, J18 Conn_01x10, J19 SW, J2 LINE_TAB, J20 SW4_TAB, J21 Conn_01x02, J22 PUMP1_TAB, J23 PUMP2_TAB, J3 Conn_01x02, J4 Conn_01x02, J5 NTC, J6 Conn_01x02, J7 JST_3P_2.54mm, J8 Conn_01x02, J9 BOILER_TAB, Q1 025N06N, Q10 025N06N, Q11 025N06N, Q12 025N06N, Q13 BT131, Q14 BT131, Q15 025N06N, Q16 BT131, Q17 BT131, Q2 025N06N, Q3 BTA16, Q4 025N06N, Q5 2N2222, Q6 025N06N, Q7 BT131, Q8 BT131, Q9 025N06N, U1 LM2596T-ADJ, U10 MOC3021M, U11 MOC3021M, U12 MOC3021M, U13 MOC3021M, U14 MOC3021M, U2 LM2596T-ADJ, U3 LM4040DBZ-3, U4 PC817, U5 PC817, U6 MOC3021M, U7 LM2596T-ADJ, U8 MOC3021M, U9 STM32F103C8Tx, Y1 Crystal_GND24

Commit message: 1
Parts:
- removed 12V, 3V3, 5V, GND: TestPoint_Pad_1.5x1.5mm, TestPoint:TestPoint_Pad_1.5x1.5mm
- U1, U2, U7: footprint Package_TO_SOT_SMD:TO-252-5_TabPin3 -> Package_TO_SOT_SMD:TO-263-5_TabPin3
- moved J21 26.3 mm to (59.2, 81.0)
- moved C2 17.7 mm to (63.3, 53.0), turned to -90 degrees
- moved C8 17.5 mm to (79.0, 52.9), turned to -90 degrees
- moved C3 17.3 mm to (94.8, 52.9), turned to -90 degrees
- moved D13 14.1 mm to (59.2, 74.5), turned to 0 degrees
- moved D3 12.1 mm to (100.9, 52.0), turned to -90 degrees
- moved D2 12.1 mm to (85.5, 52.0), turned to -90 degrees
- moved D1 11.7 mm to (109.9, 25.3)
- moved R1 11.7 mm to (109.9, 21.9)
- moved R5 11.7 mm to (104.7, 52.5), turned to 0 degrees
- moved R4 11.4 mm to (88.9, 52.4), turned to 0 degrees
- moved D12 11.2 mm to (69.6, 52.0), turned to -90 degrees
- moved R12 10.7 mm to (73.0, 52.4), turned to 0 degrees
- moved R3 10.5 mm to (104.7, 49.3), turned to 180 degrees
- moved R2 10.1 mm to (88.9, 49.3), turned to 180 degrees
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Routing:
- net +3V3: track 261.8 -> 2.85 mm, vias 4 -> 1
- net +5V: track 146.2 -> 0.00 mm, vias 1 -> 0
- net Z_CROSS: track 101.8 -> 11.9 mm, vias 2 -> 1
- net Motor_1: track 76.4 -> 1.00 mm, vias 2 -> 1
- net +24V: track 203.8 -> 132.4 mm
- net Motor_2: track 70.5 -> 1.04 mm, vias 2 -> 1
- net +12V: track 63.1 -> 0.00 mm, vias 2 -> 0
- net UART_Rx: track 39.0 -> 0.00 mm, vias 2 -> 0
- net UART_Tx: track 35.6 -> 0.00 mm, vias 2 -> 0
- net AIR_PUMP_uC: track 35.4 -> 0.00 mm, vias 2 -> 0
- net NTC: track 33.0 -> 1.50 mm
- net +3V0: track 30.7 -> 1.47 mm
- net FLOWMETER: track 21.2 -> 0.00 mm, vias 2 -> 0
- net Net-(Q15-Pad1): track 13.8 -> 0.00 mm
- net Net-(C24-Pad2): track 13.2 -> 0.00 mm
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- removed copper zone on F.Cu, net +24V
- removed copper zone on F.Cu, net Net-(C10-Pad1)
- removed copper zone on F.Cu, net Net-(C6-Pad1)
- removed copper zone on F.Cu, net Net-(C7-Pad1)
- removed copper zone on F.Cu, net Net-(D12-Pad1)
- removed copper zone on F.Cu, net Net-(D2-Pad1)
- removed copper zone on F.Cu, net Net-(D3-Pad1)
Other:
- board text added: "AIR"
- board text removed: "AIR PUMP"
- board text removed: "INDUSTRY COFFEE MACHINE"

Commit message: 1
Parts:
- moved R1 61.7 mm to (57.2, 54.0)
- moved D1 58.4 mm to (57.2, 50.6)
- moved U3 0.61 mm to (75.0, 104.5), turned to 0 degrees
Connections:
- D1 pad 1: GND -> Net-(D1-Pad1)
- D1 pad 2: Net-(D1-Pad2) -> +24V
- R1 pad 1: Net-(D1-Pad2) -> GND
- R1 pad 2: +24V -> Net-(D1-Pad1)
Routing:
- net +3V3: track 2.85 -> 256.1 mm, vias 1 -> 3
- net +5V: track 0.00 -> 140.9 mm, vias 0 -> 1
- net +24V: track 132.4 -> 234.2 mm, vias 0 -> 3
- net Z_CROSS: track 11.9 -> 103.7 mm, vias 1 -> 2
- net Motor_1: track 1.00 -> 77.6 mm, vias 1 -> 2
- net Motor_2: track 1.04 -> 67.8 mm, vias 1 -> 2
- net +12V: track 0.00 -> 62.7 mm
- net UART_Tx: track 0.00 -> 40.9 mm, vias 0 -> 2
- net UART_Rx: track 0.00 -> 37.2 mm, vias 0 -> 2
- net AIR_PUMP_uC: track 0.00 -> 33.4 mm, vias 0 -> 2
- net NTC: track 1.50 -> 23.4 mm, vias 0 -> 2
- net +3V0: track 1.47 -> 22.3 mm
- net FLOWMETER: track 0.00 -> 14.2 mm, vias 0 -> 2
- net Net-(D13-Pad2): track 0.00 -> 14.1 mm
- net Net-(C24-Pad2): track 0.00 -> 12.5 mm
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- added copper zone on F.Cu, net +24V
- added copper zone on F.Cu, net Net-(C10-Pad1)
- added copper zone on F.Cu, net Net-(C6-Pad1)
- added copper zone on F.Cu, net Net-(C7-Pad1)
- added copper zone on F.Cu, net Net-(D12-Pad1)
- added copper zone on F.Cu, net Net-(D2-Pad1)
- added copper zone on F.Cu, net Net-(D3-Pad1)
