File: Coffee_Machine_Gogokhia_Edition_SIMPLE_V1.0/PCB/DcMotorControl.kicad_sch (KiCad schematic)
At the start: 8 parts

Commit message: Edited
Parts:
- added D10, D11, D6, D7, D8, D9: D, Diode_SMD:D_SMA, symbol Device:D
- added J10, J13, J16, J17, J6, J8: Conn_01x02, Footprint:Molex_White_4_2mm_2P, symbol Connector_Generic:Conn_01x02
- added Q10, Q11, Q12, Q4, Q6, Q9: 025N06N, Package_TO_SOT_SMD:TO-252-2, symbol Transistor_FET:AO3400A
- added R10, R13, R14, R19, R20, R22: 1K, Resistor_SMD:R_0603_1608Metric, symbol Device:R
- D4, D5: renamed from D?; footprint Diode_SMD:D_SMB -> Diode_SMD:D_SMA
- J3, J4: renamed from J?; footprint (none) -> Footprint:Molex_White_4_2mm_2P
- Q1, Q2: renamed from Q?; footprint Package_TO_SOT_SMD:SOT-23 -> Package_TO_SOT_SMD:TO-252-2
- R7, R8: renamed from R?; footprint Resistor_SMD:R_0603_1608Metric_Pad1.05x0.95mm_HandSolder -> Resistor_SMD:R_0603_1608Metric
Connections:
- net +24V: now also D10.1 (K), D11.1 (K), D6.1 (K), D7.1 (K), D8.1 (K), D9.1 (K), J10.1 (Pin_1), J13.1 (Pin_1), J16.1 (Pin_1), J17.1 (Pin_1), J6.1 (Pin_1), J8.1 (Pin_1)
- net GND: now also Q10.2 (S), Q11.2 (S), Q12.2 (S), Q4.2 (S), Q6.2 (S), Q9.2 (S)
- new net: D9.2 (A), J13.2 (Pin_2), Q10.3 (D)
- new net: D8.2 (A), J10.2 (Pin_2), Q9.3 (D)
- new net: D6.2 (A), J6.2 (Pin_2), Q4.3 (D)
- new net: Q10.1 (G), R19.2
- new net: D7.2 (A), J8.2 (Pin_2), Q6.3 (D)
- new net: Q4.1 (G), R10.2
- new net: Q11.1 (G), R20.2
- new net: D10.2 (A), J16.2 (Pin_2), Q11.3 (D)
- new net: Q9.1 (G), R14.2
- new net: D11.2 (A), J17.2 (Pin_2), Q12.3 (D)
- new net: Q12.1 (G), R22.2
- new net: Q6.1 (G), R13.2
- new net Motor_3: R10.1
- new net Motor_4: R19.1
- new net Motor_5: R13.1
- new net Motor_6: R20.1
- new net Motor_7: R14.1
- new net Motor_8: R22.1
Other:
- moved on the sheet: D4, D5, J3, J4, Q1, Q2, R7, R8

Commit message: 1
Parts:
- added R27, R28, R29, R30, R31, R32, R33, R34: 10K, Resistor_SMD:R_0603_1608Metric, symbol Device:R
Connections:
- net +24V: now also J10.2 (Pin_2), J13.2 (Pin_2), J16.2 (Pin_2), J17.2 (Pin_2), J3.2 (Pin_2), J4.2 (Pin_2), J6.2 (Pin_2), J8.2 (Pin_2); no longer J10.1 (Pin_1), J13.1 (Pin_1), J16.1 (Pin_1), J17.1 (Pin_1), J3.1 (Pin_1), J4.1 (Pin_1), J6.1 (Pin_1), J8.1 (Pin_1)
- net GND: now also R27.2, R28.2, R29.2, R30.2, R31.2, R32.2, R33.2, R34.2
- net at D9.2 (A), Q10.3 (D): now also J13.1 (Pin_1); no longer J13.2 (Pin_2)
- net at Q1.1 (G), R7.2: now also R29.1
- net at D4.2 (A), Q1.3 (D): now also J3.1 (Pin_1); no longer J3.2 (Pin_2)
- net at D8.2 (A), Q9.3 (D): now also J10.1 (Pin_1); no longer J10.2 (Pin_2)
- net at D6.2 (A), Q4.3 (D): now also J6.1 (Pin_1); no longer J6.2 (Pin_2)
- net at Q2.1 (G), R8.2: now also R34.1
- net at D5.2 (A), Q2.3 (D): now also J4.1 (Pin_1); no longer J4.2 (Pin_2)
- net at Q10.1 (G), R19.2: now also R31.1
- net at D7.2 (A), Q6.3 (D): now also J8.1 (Pin_1); no longer J8.2 (Pin_2)
- net at Q4.1 (G), R10.2: now also R30.1
- net at Q11.1 (G), R20.2: now also R32.1
- net at D10.2 (A), Q11.3 (D): now also J16.1 (Pin_1); no longer J16.2 (Pin_2)
- net at Q9.1 (G), R14.2: now also R28.1
- net at D11.2 (A), Q12.3 (D): now also J17.1 (Pin_1); no longer J17.2 (Pin_2)
- net at Q12.1 (G), R22.2: now also R33.1
- net at Q6.1 (G), R13.2: now also R27.1
