File: Coffee_Machine_Gogokhia_Edition_SIMPLE_V1.0/PCB/NTC.kicad_sch (KiCad schematic)
At the start: 6 parts

Commit message: Edited
Parts:
- removed C?: .01uF, Capacitor_SMD:C_0603_1608Metric, symbol Device:C
- removed J?: NTC, Connector_JST:JST_EH_B2B-EH-A_1x02_P2.50mm_Vertical, symbol Connector_Generic:Conn_01x02
- removed R?: 47K, Resistor_SMD:R_0603_1608Metric, symbol Device:R
- J5: renamed from J?; footprint Connector_JST:JST_EH_B2B-EH-A_1x02_P2.50mm_Vertical -> Footprint:JST_2.54_2P
- gave numbers to parts that had none: 2
Other:
- note removed: "NTC_Cap"
Changed lines of the file:
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@@
   (junction (at 115.57 87.63) (diameter 0) (color 0 0 0 0)
-  )
-  (junction (at 158.75 87.63) (diameter 0) (color 0 0 0 0)
   )
   (junction (at 115.57 96.52) (diameter 0) (color 0 0 0 0)
@@
   (junction (at 120.65 87.63) (diameter 0) (color 0 0 0 0)
   )
-  (junction (at 153.67 87.63) (diameter 0) (color 0 0 0 0)
-  )
-  (junction (at 153.67 96.52) (diameter 0) (color 0 0 0 0)
-  )
   (polyline (pts (xy 135.89 101.6) (xy 104.14 101.6))
     (stroke (width 0) (type default) (color 0 0 0 0))
   )
-  (wire (pts (xy 158.75 96.52) (xy 158.75 95.25))
-    (stroke (width 0) (type default) (color 0 0 0 0))
-  )
   (wire (pts (xy 115.57 77.47) (xy 115.57 76.2))
-    (stroke (width 0) (type default) (color 0 0 0 0))
-  )
-  (wire (pts (xy 153.67 92.71) (xy 151.13 92.71))
-    (stroke (width 0) (type default) (color 0 0 0 0))
-  )
-  (wire (pts (xy 153.67 87.63) (xy 153.67 85.09))
     (stroke (width 0) (type default) (color 0 0 0 0))
   )
@@
     (stroke (width 0) (type default) (color 0 0 0 0))
   )
-  (wire (pts (xy 153.67 96.52) (xy 153.67 97.79))
-    (stroke (width 0) (type default) (color 0 0 0 0))
-  )
   (wire (pts (xy 115.57 90.17) (xy 115.57 87.63))
-    (stroke (width 0) (type default) (color 0 0 0 0))
-  )
-  (wire (pts (xy 153.67 77.47) (xy 153.67 76.2))
-    (stroke (width 0) (type default) (color 0 0 0 0))
-  )
-  (wire (pts (xy 153.67 92.71) (xy 153.67 96.52))
     (stroke (width 0) (type default) (color 0 0 0 0))
   )
@@
     (stroke (width 0) (type default) (color 0 0 0 0))
   )
-  (wire (pts (xy 167.64 87.63) (xy 158.75 87.63))
-    (stroke (width 0) (type default) (color 0 0 0 0))
-  )
-  (wire (pts (xy 153.67 96.52) (xy 158.75 96.52))
-    (stroke (width 0) (type default) (color 0 0 0 0))
-  )
-  (polyline (pts (xy 142.24 69.85) (xy 179.07 69.85))
-    (stroke (width 0) (type default) (color 0 0 0 0))
-  )
-  (wire (pts (xy 153.67 87.63) (xy 158.75 87.63))
-    (stroke (width 0) (type default) (color 0 0 0 0))
-  )
   (wire (pts (xy 115.57 87.63) (xy 115.57 85.09))
     (stroke (width 0) (type default) (color 0 0 0 0))
@@
     (stroke (width 0) (type default) (color 0 0 0 0))
   )
-  (wire (pts (xy 153.67 90.17) (xy 153.67 87.63))
-    (stroke (width 0) (type default) (color 0 0 0 0))
-  )
-  (polyline (pts (xy 142.24 101.6) (xy 142.24 69.85))
-    (stroke (width 0) (type default) (color 0 0 0 0))
-  )
-  (polyline (pts (xy 179.07 69.85) (xy 179.07 101.6))
-    (stroke (width 0) (type default) (color 0 0 0 0))
-  )
-  (polyline (pts (xy 179.07 101.6) (xy 142.24 101.6))
-    (stroke (width 0) (type default) (color 0 0 0 0))
-  )
   (wire (pts (xy 115.57 87.63) (xy 120.65 87.63))
     (stroke (width 0) (type default) (color 0 0 0 0))
   )
-  (wire (pts (xy 151.13 90.17) (xy 153.67 90.17))
-    (stroke (width 0) (type default) (color 0 0 0 0))
-  )
   (text "NTC" (at 130.81 72.39 0)
-    (effects (font (size 1.27 1.27)) (justify left bottom))
-  )
-  (text "NTC_Cap" (at 163.83 72.39 0)
     (effects (font (size 1.27 1.27)) (justify left bottom))
   )
@@
     )
   )
-  (global_label "NTC_Cap" (shape input) (at 167.64 87.63 0) (fields_autoplaced)
-    (effects (font (size 1.27 1.27)) (justify left))
-    (property "Intersheet References" "${INTERSHEET_REFS}" (id 0) (at 178.068 87.5506 0)
-      (effects (font (size 1.27 1.27)) (justify left) hide)
-    )
-  )
   (symbol (lib_id "Connector_Generic:Conn_01x02") (at 107.95 90.17 0) (mirror y) (unit 1)
     (in_bom yes) (on_board yes)
-    (property "Reference" "J?" (id 0) (at 105.918 90.3732 0)
+    (property "Reference" "J5" (id 0) (at 105.918 90.3732 0)
       (effects (font (size 1.27 1.27)) (justify left) hide)
     )
     (property "Value" "NTC" (id 1) (at 105.41 91.44 90))
-    (property "Footprint" "Connector_JST:JST_EH_B2B-EH-A_1x02_P2.50mm_Vertical" (id 2) (at 107.95 90.17 0)
+    (property "Footprint" "Footprint:JST_2.54_2P" (id 2) (at 107.95 90.17 0)
       (effects (font (size 1.27 1.27)) hide)
     )
@@
   (symbol (lib_id "power:GND") (at 115.57 97.79 0) (unit 1)
     (in_bom yes) (on_board yes)
-    (property "Reference" "#PWR?" (id 0) (at 115.57 104.14 0)
+    (property "Reference" "#PWR0131" (id 0) (at 115.57 104.14 0)
       (effects (font (size 1.27 1.27)) hide)
     )
@@
     (pin "1")
   )
-  (symbol (lib_id "Connector_Generic:Conn_01x02") (at 146.05 90.17 0) (mirror y) (unit 1)
-    (in_bom yes) (on_board yes)
-    (property "Reference" "J?" (id 0) (at 144.018 90.3732 0)
-      (effects (font (size 1.27 1.27)) (justify left) hide)
-    )
-    (property "Value" "NTC" (id 1) (at 143.51 91.44 90))
-    (property "Footprint" "Connector_JST:JST_EH_B2B-EH-A_1x02_P2.50mm_Vertical" (id 2) (at 146.05 90.17 0)
-      (effects (font (size 1.27 1.27)) hide)
-    )
-    (property "Datasheet" "~" (id 3) (at 146.05 90.17 0)
-      (effects (font (size 1.27 1.27)) hide)
-    )
-    (pin "1")
-    (pin "2")
-  )
-  (symbol (lib_id "Device:C") (at 158.75 91.44 0) (unit 1)
-    (in_bom yes) (on_board yes)
-    (property "Reference" "C?" (id 0) (at 161.671 90.2716 0)
-      (effects (font (size 1.27 1.27)) (justify left))
-    )
-    (property "Value" ".01uF" (id 1) (at 161.671 92.583 0)
-      (effects (font (size 1.27 1.27)) (justify left))
-    )
-    (property "Footprint" "Capacitor_SMD:C_0603_1608Metric" (id 2) (at 159.7152 95.25 0)
-      (effects (font (size 1.27 1.27)) hide)
-    )
-    (property "Datasheet" "~" (id 3) (at 158.75 91.44 0)
-      (effects (font (size 1.27 1.27)) hide)
-    )
-    (pin "1")
-    (pin "2")
-  )
   (symbol (lib_id "Device:R") (at 115.57 81.28 0) (unit 1)
     (in_bom yes) (on_board yes)
-    (property "Reference" "R?" (id 0) (at 118.11 81.28 90))
+    (property "Reference" "R9" (id 0) (at 118.11 81.28 90))
     (property "Value" "47K" (id 1) (at 115.57 81.28 90))
     (property "Footprint" "Resistor_SMD:R_0603_1608Metric" (id 2) (at 113.792 81.28 90)
@@
   (symbol (lib_id "power:+3V0") (at 115.57 76.2 0) (unit 1)
     (in_bom yes) (on_board yes)
-    (property "Reference" "#PWR?" (id 0) (at 115.57 80.01 0)
+    (property "Reference" "#PWR0130" (id 0) (at 115.57 80.01 0)
       (effects (font (size 1.27 1.27)) hide)
     )
@@
     (pin "1")
   )
-  (symbol (lib_id "Device:R") (at 153.67 81.28 0) (unit 1)
-    (in_bom yes) (on_board yes)
-    (property "Reference" "R?" (id 0) (at 156.21 81.28 90))
-    (property "Value" "47K" (id 1) (at 153.67 81.28 90))
-    (property "Footprint" "Resistor_SMD:R_0603_1608Metric" (id 2) (at 151.892 81.28 90)
-      (effects (font (size 1.27 1.27)) hide)
-    )
-    (property "Datasheet" "~" (id 3) (at 153.67 81.28 0)
-      (effects (font (size 1.27 1.27)) hide)
-    )
-    (pin "1")
-    (pin "2")
-  )
-  (symbol (lib_id "power:+3V0") (at 153.67 76.2 0) (unit 1)
-    (in_bom yes) (on_board yes)
-    (property "Reference" "#PWR?" (id 0) (at 153.67 80.01 0)
-      (effects (font (size 1.27 1.27)) hide)
-    )
-    (property "Value" "+3V0" (id 1) (at 154.051 71.8058 0))
-    (property "Footprint" "" (id 2) (at 153.67 76.2 0)
-      (effects (font (size 1.27 1.27)) hide)
-    )
-    (property "Datasheet" "" (id 3) (at 153.67 76.2 0)
-      (effects (font (size 1.27 1.27)) hide)
-    )
-    (pin "1")
-  )
   (symbol (lib_id "Device:C") (at 120.65 91.44 0) (unit 1)
     (in_bom yes) (on_board yes)
-    (property "Reference" "C?" (id 0) (at 123.571 90.2716 0)
+    (property "Reference" "C27" (id 0) (at 123.571 90.2716 0)
       (effects (font (size 1.27 1.27)) (justify left))
     )
@@
     (pin "2")
   )
-  (symbol (lib_id "power:GND") (at 153.67 97.79 0) (unit 1)
-    (in_bom yes) (on_board yes)
-    (property "Reference" "#PWR?" (id 0) (at 153.67 104.14 0)
-      (effects (font (size 1.27 1.27)) hide)
-    )
-    (property "Value" "GND" (id 1) (at 153.797 102.1842 0)
-      (effects (font (size 1.27 1.27)) hide)
-    )
-    (property "Footprint" "" (id 2) (at 153.67 97.79 0)
-      (effects (font (size 1.27 1.27)) hide)
-    )
-    (property "Datasheet" "" (id 3) (at 153.67 97.79 0)
-      (effects (font (size 1.27 1.27)) hide)
-    )
-    (pin "1")
-  )
 )

Commit message: 1
Parts:
- R9: value 47K -> 100K
Changed lines of the file:
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@@
     (in_bom yes) (on_board yes)
     (property "Reference" "R9" (id 0) (at 118.11 81.28 90))
-    (property "Value" "47K" (id 1) (at 115.57 81.28 90))
+    (property "Value" "100K" (id 1) (at 115.57 81.28 90))
     (property "Footprint" "Resistor_SMD:R_0603_1608Metric" (id 2) (at 113.792 81.28 90)
       (effects (font (size 1.27 1.27)) hide)
