File: Coffee_Machine_Gogokhia_Edition_SIMPLE_V1.0/PCB/Pump.kicad_sch (KiCad schematic)
At the start: 16 parts

Commit message: Edited
Parts:
- removed C?: .01uF, Capacitor_THT:C_Disc_D4.7mm_W2.5mm_P5.00mm, symbol Device:C
- removed J?: PUMP_TAB_Cap, MyLibrary:TAB_CONN, symbol Connector:Conn_01x01_Male
- removed Q?: BT131, MyLibrary:TO127P254X732-3, symbol Triac_Thyristor:BTA16-600B
- removed R?: 180R, Resistor_SMD:R_1206_3216Metric, symbol Device:R
- removed R?: 10K, Resistor_SMD:R_0603_1608Metric, symbol Device:R
- removed R?: 330R, Resistor_SMD:R_0603_1608Metric, symbol Device:R
- removed R?: 39R, Resistor_SMD:R_1206_3216Metric, symbol Device:R
- removed U?: MOC3021M, MyLibrary:OPTOCOUPLER_H11F3SR2M, symbol Relay_SolidState:MOC3021M
- C35: renamed from C?; footprint Capacitor_THT:C_Disc_D4.7mm_W2.5mm_P5.00mm -> Capacitor_THT:C_Disc_D5.0mm_W2.5mm_P5.00mm
- J12: renamed from J?; footprint MyLibrary:TAB_CONN -> Footprint:TAB_Conn
- Q5: renamed from Q?; footprint MyLibrary:TO127P254X732-3 -> Footprint:BT131
- U8: renamed from U?; footprint MyLibrary:OPTOCOUPLER_H11F3SR2M -> Footprint:DIP6_SMD
- gave numbers to parts that had none: 4
Other:
- note removed: "PUMP_Cap"

Commit message: 1
Parts:
- removed C35: .01uF, Capacitor_THT:C_Disc_D5.0mm_W2.5mm_P5.00mm, symbol Device:C
- removed J12: PUMP_TAB, Footprint:TAB_Conn, symbol Connector:Conn_01x01_Male
- removed Q5: BT131, Footprint:BT131, symbol Triac_Thyristor:BTA16-600B
- removed R27: 330R, Resistor_SMD:R_0603_1608Metric, symbol Device:R
- removed R29: 10K, Resistor_SMD:R_0603_1608Metric, symbol Device:R
- removed R31: 180R, Resistor_SMD:R_1206_3216Metric, symbol Device:R
- removed R33: 39R, Resistor_SMD:R_1206_3216Metric, symbol Device:R
- removed U8: MOC3021M, Footprint:DIP6_SMD, symbol Relay_SolidState:MOC3021M
- added D13: D, Diode_SMD:D_SMA, symbol Device:D
- added J21: Conn_01x02, Footprint:JST_2.54_2P, symbol Connector_Generic:Conn_01x02
- added Q15: 025N06N, Package_TO_SOT_SMD:TO-252-2, symbol Transistor_FET:AO3400A
- added R55: 1K, Resistor_SMD:R_0603_1608Metric, symbol Device:R
- added R56: 10K, Resistor_SMD:R_0603_1608Metric, symbol Device:R
Connections:
- net GND: now also Q15.2 (S), R56.2
- new net: D13.2 (A), J21.1 (Pin_1), Q15.3 (D)
- new net: Q15.1 (G), R55.2, R56.1
- new net +12V: D13.1 (K), J21.2 (Pin_2)
- new net AIR_PUMP_uC: R55.1
Other:
- note added: "AIR PUMP"
- note removed: "PUMP"
