File: Coffee_Machine_Gogokhia_Edition_SIMPLE_V1.0/PCB/ZeroCross.kicad_sch (KiCad schematic)
At the start: 4 parts

Commit message: Edited
Parts:
- R15: renamed from R?; footprint Resistor_SMD:R_0603_1608Metric -> Resistor_SMD:R_1206_3216Metric
- U4, U5: renamed from U?; footprint MyLibrary:SOT254P975X400-4N -> Footprint:PC817
- gave numbers to parts that had none: 1
Changed lines of the file:
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@@
   (symbol (lib_id "power:GND") (at 139.7 93.98 0) (unit 1)
     (in_bom yes) (on_board yes)
-    (property "Reference" "#PWR?" (id 0) (at 139.7 100.33 0)
+    (property "Reference" "#PWR0144" (id 0) (at 139.7 100.33 0)
       (effects (font (size 1.27 1.27)) hide)
     )
@@
   (symbol (lib_id "power:GND") (at 139.7 107.95 0) (unit 1)
     (in_bom yes) (on_board yes)
-    (property "Reference" "#PWR?" (id 0) (at 139.7 114.3 0)
+    (property "Reference" "#PWR0143" (id 0) (at 139.7 114.3 0)
       (effects (font (size 1.27 1.27)) hide)
     )
@@
   (symbol (lib_id "power:+3V3") (at 142.24 76.2 0) (unit 1)
     (in_bom yes) (on_board yes)
-    (property "Reference" "#PWR?" (id 0) (at 142.24 80.01 0)
+    (property "Reference" "#PWR0142" (id 0) (at 142.24 80.01 0)
       (effects (font (size 1.27 1.27)) hide)
     )
@@
   (symbol (lib_id "Isolator:PC817") (at 129.54 88.9 0) (unit 1)
     (in_bom yes) (on_board yes)
-    (property "Reference" "U?" (id 0) (at 129.54 80.645 0))
+    (property "Reference" "U4" (id 0) (at 129.54 80.645 0))
     (property "Value" "PC817" (id 1) (at 129.54 82.9564 0))
-    (property "Footprint" "MyLibrary:SOT254P975X400-4N" (id 2) (at 124.46 93.98 0)
+    (property "Footprint" "Footprint:PC817" (id 2) (at 124.46 93.98 0)
       (effects (font (size 1.27 1.27) italic) (justify left) hide)
     )
@@
   (symbol (lib_id "Device:R") (at 142.24 81.28 180) (unit 1)
     (in_bom yes) (on_board yes)
-    (property "Reference" "R?" (id 0) (at 144.78 81.28 90))
+    (property "Reference" "R16" (id 0) (at 144.78 81.28 90))
     (property "Value" "10K" (id 1) (at 142.24 81.28 90))
     (property "Footprint" "Resistor_SMD:R_0603_1608Metric" (id 2) (at 144.018 81.28 90)
@@
   (symbol (lib_id "Device:R") (at 115.57 86.36 270) (unit 1)
     (in_bom yes) (on_board yes)
-    (property "Reference" "R?" (id 0) (at 115.57 83.82 90))
+    (property "Reference" "R15" (id 0) (at 115.57 83.82 90))
     (property "Value" "100K" (id 1) (at 115.57 86.36 90))
-    (property "Footprint" "Resistor_SMD:R_0603_1608Metric" (id 2) (at 115.57 84.582 90)
+    (property "Footprint" "Resistor_SMD:R_1206_3216Metric" (id 2) (at 115.57 84.582 90)
       (effects (font (size 1.27 1.27)) hide)
     )
@@
   (symbol (lib_id "Isolator:PC817") (at 129.54 102.87 0) (unit 1)
     (in_bom yes) (on_board yes)
-    (property "Reference" "U?" (id 0) (at 129.54 94.615 0))
+    (property "Reference" "U5" (id 0) (at 129.54 94.615 0))
     (property "Value" "PC817" (id 1) (at 129.54 96.9264 0))
-    (property "Footprint" "MyLibrary:SOT254P975X400-4N" (id 2) (at 124.46 107.95 0)
+    (property "Footprint" "Footprint:PC817" (id 2) (at 124.46 107.95 0)
       (effects (font (size 1.27 1.27) italic) (justify left) hide)
     )

Commit message: 1
Changed lines of the file:
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@@
     (stroke (width 0) (type default) (color 0 0 0 0))
   )
-  (text "ZERO CROSS\n" (at 119.38 49.53 0)
+  (text "ZERO CROSS\n" (at 106.68 65.659 0)
     (effects (font (size 3 3)) (justify left bottom))
   )
