File: Coffee_Machine_Gogokhia_Edition_SIMPLE_V1.0/PCB/eValve.kicad_sch (KiCad schematic)
At the start: 32 parts

Commit message: Edited
Parts:
- removed C? (x2): .01uF, Capacitor_THT:C_Disc_D5.0mm_W2.5mm_P5.00mm, symbol Device:C
- removed J?: SW1_TAB_Cap, MyLibrary:TAB_CONN, symbol Connector:Conn_01x01_Male
- removed J?: SW2_TAB_Cap, MyLibrary:TAB_CONN, symbol Connector:Conn_01x01_Male
- removed Q? (x2): BT131, MyLibrary:TO127P254X732-3, symbol Triac_Thyristor:BTA16-600B
- removed R? (x2): 180R, Resistor_SMD:R_1206_3216Metric, symbol Device:R
- removed R? (x2): 39R, Resistor_SMD:R_1206_3216Metric, symbol Device:R
- removed R? (x2): 10K, Resistor_SMD:R_0603_1608Metric, symbol Device:R
- removed R? (x2): 330R, Resistor_SMD:R_0603_1608Metric, symbol Device:R
- removed U? (x2): MOC3021M, MyLibrary:OPTOCOUPLER_H11F3SR2M, symbol Relay_SolidState:MOC3021M
- J14, J15: renamed from J?; footprint MyLibrary:TAB_CONN -> Footprint:TAB_Conn
- Q7, Q8: renamed from Q?; footprint MyLibrary:TO127P254X732-3 -> Footprint:BT131
- U11, U12: renamed from U?; footprint MyLibrary:OPTOCOUPLER_H11F3SR2M -> Footprint:DIP6_SMD
- gave numbers to parts that had none: 10
Other:
- note removed: "SW_Cap_1"
- note removed: "SW_Cap_2"

Commit message: 1
Parts:
- added C29, C30: .01uF, Capacitor_THT:C_Disc_D5.0mm_W2.5mm_P5.00mm, symbol Device:C
- added J12: SW3_TAB, Footprint:TAB_Conn, symbol Connector:Conn_01x01_Male
- added J20: SW4_TAB, Footprint:TAB_Conn, symbol Connector:Conn_01x01_Male
- added Q13, Q14: BT131, Footprint:BT131, symbol Triac_Thyristor:BTA16-600B
- added R47, R48: 330R, Resistor_SMD:R_0603_1608Metric, symbol Device:R
- added R49, R50: 10K, Resistor_SMD:R_0603_1608Metric, symbol Device:R
- added R51, R52: 180R, Resistor_SMD:R_1206_3216Metric, symbol Device:R
- added R53, R54: 39R, Resistor_SMD:R_1206_3216Metric, symbol Device:R
- added U10, U8: MOC3021M, Footprint:DIP6_SMD, symbol Relay_SolidState:MOC3021M
Connections:
- net GND: now also R49.1, R50.1, U10.2, U8.2
- net LINE: now also Q13.1 (A1), Q14.1 (A1), R53.1, R54.1
- new net: R48.1, R50.2, U10.1
- new net: R47.1, R49.2, U8.1
- new net: C30.1, J20.1 (Pin_1), Q14.2 (A2), R52.1
- new net: Q14.3 (G), U10.4
- new net: R52.2, U10.6
- new net: C29.1, J12.1 (Pin_1), Q13.2 (A2), R51.1
- new net: Q13.3 (G), U8.4
- new net: C29.2, R53.2
- new net: C30.2, R54.2
- new net: R51.2, U8.6
- new net SW3_uC: R47.2
- new net SW4_uC: R48.2
Other:
- note added: "SW 3"
- note added: "SW 4"
