File: Coffee_Machine_Gogokhia_Edition_SIMPLE_V1.0/PCB/Coffe_Machine_Gogokhia_Edition_SIMPLE.kicad_sch (KiCad schematic)
At the start: 142 parts, among them J1 LINE_TAB, J11 SW, J2 NEUT_TAB, J3 NTC, J4 BOILER_TAB, J5 PUMP_TAB, J6 SW1_TAB, J7 SW2_TAB, J8 FLOWMETER, Q1 BTA16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

Commit message: update
Parts:
- removed C1, C3, C4, C? (x3): .01uF, Capacitor_THT:C_Disc_D5.0mm_W2.5mm_P5.00mm, symbol Device:C
- removed C2, C?: .01uF, Capacitor_THT:C_Disc_D4.7mm_W2.5mm_P5.00mm, symbol Device:C
- removed C5, C9, C? (x2): .01uF, Capacitor_SMD:C_0603_1608Metric, symbol Device:C
- removed C7, C?: .1uF, Capacitor_SMD:C_0603_1608Metric, symbol Device:C
- removed C? (x2): 0.1uF, Capacitor_SMD:C_0603_1608Metric_Pad1.05x0.95mm_HandSolder, symbol Device:C
- removed C? (x2): 0.01uF, Capacitor_SMD:C_0603_1608Metric_Pad1.05x0.95mm_HandSolder, symbol Device:C
- removed C? (x2): 100uF, Capacitor_Tantalum_SMD:CP_EIA-3216-10_Kemet-I, symbol Device:CP
- removed C? (x2): 220uF, Capacitor_SMD:CP_Elec_10x10.5, symbol Device:CP
- removed C? (x2): 100uF, Capacitor_SMD:CP_Elec_10x10.5, symbol Device:CP
- removed C? (x2): 15nF, Capacitor_SMD:C_0603_1608Metric_Pad1.05x0.95mm_HandSolder, symbol Device:C
- removed D6: LED, LED_SMD:LED_0603_1608Metric, symbol Device:LED
- removed D? (x4): D, Diode_SMD:D_SMB, symbol Device:D
- removed J1: LINE_TAB, MyLibrary:TAB_CONN, symbol Connector:Conn_01x01_Male
- removed J2: NEUT_TAB, MyLibrary:TAB_CONN, symbol Connector:Conn_01x01_Male
- removed J3, J?: NTC, Connector_JST:JST_EH_B2B-EH-A_1x02_P2.50mm_Vertical, symbol Connector_Generic:Conn_01x02
- removed J4: BOILER_TAB, MyLibrary:TAB_CONN, symbol Connector:Conn_01x01_Male
- removed J5: PUMP_TAB, MyLibrary:TAB_CONN, symbol Connector:Conn_01x01_Male
- removed J6: SW1_TAB, MyLibrary:TAB_CONN, symbol Connector:Conn_01x01_Male
- removed J7: SW2_TAB, MyLibrary:TAB_CONN, symbol Connector:Conn_01x01_Male
- removed J8, J?: FLOWMETER, Connector_JST:JST_EH_B3B-EH-A_1x03_P2.50mm_Vertical, symbol Connector_Generic:Conn_01x03
- removed J?: SW2_TAB_Cap, MyLibrary:TAB_CONN, symbol Connector:Conn_01x01_Male
- removed J?: PUMP_TAB_Cap, MyLibrary:TAB_CONN, symbol Connector:Conn_01x01_Male
- removed J? (x2): Conn_01x02, symbol Connector_Generic:Conn_01x02
- removed J?: SW, Connector_PinHeader_1.27mm:PinHeader_1x04_P1.27mm_Vertical, symbol Connector_Generic:Conn_01x04
- removed J?: SW1_TAB_Cap, MyLibrary:TAB_CONN, symbol Connector:Conn_01x01_Male
- removed J?: BOILER_TAB_Cap, MyLibrary:TAB_CONN, symbol Connector:Conn_01x01_Male
- removed L? (x2): L, MyLibrary:SRR1208-470YL, symbol Device:L
- removed PS1: HLK-PM01, Footprint:IRM-90-24, symbol Converter_ACDC:HLK-PM01
- removed Q1, Q?: BTA16, Package_TO_SOT_THT:TO-220-3_Vertical, symbol Triac_Thyristor:BTA16-600B
- removed Q2, Q3, Q4, Q? (x3): BT131, MyLibrary:TO127P254X732-3, symbol Triac_Thyristor:BTA16-600B
- removed Q? (x2): 025N06N, Package_TO_SOT_SMD:SOT-23, symbol Transistor_FET:AO3400A
- removed R1: 100K, Resistor_SMD:R_0603_1608Metric, symbol Device:R
- removed R10, R21, R6, R7, R8, R9, R? (x5): 10K, Resistor_SMD:R_0603_1608Metric, symbol Device:R
- removed R11, R12, R13, R14, R? (x4): 180R, Resistor_SMD:R_1206_3216Metric, symbol Device:R
- removed R15, R?: 47K, Resistor_SMD:R_0603_1608Metric, symbol Device:R
- removed R16, R17, R18, R19, R? (x4): 39R, Resistor_SMD:R_1206_3216Metric, symbol Device:R
- removed R2, R3, R4, R5, R? (x4): 330R, Resistor_SMD:R_0603_1608Metric, symbol Device:R
- removed R20: 33R, Resistor_SMD:R_0603_1608Metric, symbol Device:R
- removed R22, R?: 1K, Resistor_SMD:R_0603_1608Metric, symbol Device:R
- removed R32: 4.1K, Resistor_SMD:R_0603_1608Metric, symbol Device:R
- removed R?: 20k, Resistor_SMD:R_0603_1608Metric_Pad1.05x0.95mm_HandSolder, symbol Device:R
- removed R? (x4): 1K, Resistor_SMD:R_0603_1608Metric_Pad1.05x0.95mm_HandSolder, symbol Device:R
- removed R?: 3K, Resistor_SMD:R_0603_1608Metric_Pad1.05x0.95mm_HandSolder, symbol Device:R
- removed R?: 1.6K, Resistor_SMD:R_0603_1608Metric_Pad1.05x0.95mm_HandSolder, symbol Device:R
- removed R?: 10k, Resistor_SMD:R_0603_1608Metric_Pad1.05x0.95mm_HandSolder, symbol Device:R
- removed U1, U2: PC817, MyLibrary:SOT254P975X400-4N, symbol Isolator:PC817
- removed U3, U4, U5, U6, U? (x4): MOC3021M, MyLibrary:OPTOCOUPLER_H11F3SR2M, symbol Relay_SolidState:MOC3021M
- removed U8: LM4040DBZ-3, Package_TO_SOT_SMD:SOT-23, symbol Reference_Voltage:LM4040DBZ-3
- removed U? (x2): LM2596T-ADJ, Package_TO_SOT_SMD:TO-263-5_TabPin3, symbol Regulator_Switching:LM2596T-ADJ
Other:
- added sheet Boiler (Boiler.kicad_sch)
- added sheet Dc Motor Control (DcMotorControl.kicad_sch)
- added sheet Display (Display.kicad_sch)
- added sheet Flowmeter (Flowmeter.kicad_sch)
- added sheet NTC (NTC.kicad_sch)
- added sheet Power (Power.kicad_sch)
- added sheet Pump (Pump.kicad_sch)
- added sheet ZeroCross (ZeroCross.kicad_sch)
- added sheet eValve (eValve.kicad_sch)
- note removed: "3.3V"
- note removed: "5V"
- note removed: "BOILER"
- note removed: "BOILER_Cap"
- note removed: "DC motor driver"
- note removed: "Display"
- note removed: "FLOWMETER"
- note removed: "FLOWMETER For Cap"
- note removed: "NTC"
- note removed: "NTC_Cap"
- note removed: "POWER SUPPLY"
- note removed: "PUMP"
- note removed: "PUMP_Cap"
- note removed: "SW 1"
- note removed: "SW 2"
- note removed: "SW_Cap_1"
- note removed: "SW_Cap_2"
- note removed: "ZERO CROSS"
- moved on the sheet: C11, C12, C13, C14, C15, C16, C17, C18, C19, C20, C21, C22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

Commit message: 1
Other:
- moved on the sheet: C11, C12, C13, C14, C15, C16, C17, C18, C19, C20, C21, C22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

Commit message: Edited
Parts:
- removed C20: CP, Capacitor_THT:CP_Radial_D6.3mm_P2.50mm, symbol Device:CP
- J11: footprint Connector_PinHeader_1.27mm:PinHeader_1x04_P1.27mm_Vertical -> Connector_PinSocket_1.27mm:PinSocket_1x04_P1.27mm_Vertical
- Y1: footprint Crystal:Crystal_SMD_3225-4Pin_3.2x2.5mm_HandSoldering -> Footprint:Crystal_smd_3225
Connections:
- net BOILER_uC_Cap is gone; now on net BOILER_uC: U9.21 (PB10)
- net BOILER_uC: no longer U9.40 (PB4)
- net Motor_1: now also U9.4 (PC15); no longer U9.10 (PA0)
- net Motor_2: now also U9.10 (PA0); no longer U9.11 (PA1)
- net PUMP_uC: now also U9.20 (PB2); no longer U9.42 (PB6)
- net SW1_uC: now also U9.18 (PB0); no longer U9.14 (PA4)
- net SW2_uC: now also U9.19 (PB1); no longer U9.15 (PA5)
- net Motor_7: now reaches U9.16 (PA6)
- net DC: no longer names the net of U9.22 (PB11)
- net FLOWMETER_Cap: no longer names the net of U9.32 (PA11)
- net NTC_Cap renamed Motor_4
- net PUMP_uC_Cap: no longer names the net of U9.46 (PB9)
- net RES renamed Motor_8
- net SCREEN_LED: no longer names the net of U9.29 (PA8)
- net SPI2_CS_SCREEN: no longer names the net of U9.25 (PB12)
- net SPI2_MISO: no longer names the net of U9.27 (PB14)
- net SPI2_MOSI: no longer names the net of U9.28 (PB15)
- net SPI2_SCK: no longer names the net of U9.26 (PB13)
- net SW1_uC_Cap: no longer names the net of U9.45 (PB8)
- net SW2_uC_Cap: no longer names the net of U9.43 (PB7)
- new net Motor_3: U9.11 (PA1)
- new net Motor_5: U9.14 (PA4)
- new net Motor_6: U9.15 (PA5)

Commit message: 1
Connections:
- net PUMP_uC is gone; now on net BOILER_uC: U9.20 (PB2)
- net BOILER_uC: no longer U9.21 (PB10)
- net Motor_1: now also U9.32 (PA11); no longer U9.4 (PC15)
- net Motor_2: now also U9.29 (PA8); no longer U9.10 (PA0)
- net Motor_3: now also U9.28 (PB15); no longer U9.11 (PA1)
- net Motor_4: now also U9.27 (PB14); no longer U9.12 (PA2)
- net Motor_5: now also U9.26 (PB13); no longer U9.14 (PA4)
- net Motor_6: now also U9.25 (PB12); no longer U9.15 (PA5)
- net Motor_7: now also U9.21 (PB10); no longer U9.16 (PA6)
- net Motor_8: now also U9.22 (PB11); no longer U9.17 (PA7)
- net SW1_uC: now also U9.17 (PA7); no longer U9.18 (PB0)
- net SW2_uC: now also U9.16 (PA6); no longer U9.19 (PB1)
- net AIR_PUMP_uC: now reaches U9.42 (PB6)
- net OSC_IN: no longer names the net of C15.2, U9.5 (PD0), Y1.1
- net OSC_OUT: no longer names the net of C16.2, U9.6 (PD1), Y1.3
- new net PUMP1_uC: U9.19 (PB1)
- new net PUMP2_uC: U9.18 (PB0)
- new net SW3_uC: U9.15 (PA5)
- new net SW4_uC: U9.14 (PA4)
Other:
- removed sheet Pump
- added sheet AirPump (Pump.kicad_sch)
- added sheet PUMP (untitled.kicad_sch)
- note added: "+ 1 PUMP and + 1 Valve"
- note added: "100KOhm REsistor in series AT NTC"
- note added: "AIR PUMP +12V"
- note added: "FLOWMETER CHANGE to LVL SHIFTER SCHEME"
- note added: "MOSFET on 24V MOTORS CHECK"
- note added: "Power Supply 12V"
- moved on the sheet: C15, C16, C18, R24, Y1
