File: Coffee_Machine_Gogokhia_Edition_SIMPLE_V1.0/PCB/Power.kicad_sch (KiCad schematic)
At the start: 29 parts

Commit message: 1
Other:
- note added: "#What's the inductance?"
- note added: "Put filter Capacitor between L and N. also PPTC fuse and varistor"
- note added: "Which diode?"
- note added: "Which one?"
Changed lines of the file:
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@@
     (stroke (width 0) (type default) (color 0 0 0 0))
+  )
+  (text "Which one?" (at 244.983 114.3 180)
+    (effects (font (size 1.27 1.27) (thickness 0.254) bold) (justify right bottom))
   )
   (text "5V" (at 123.19 42.545 0)
     (effects (font (size 2 2)) (justify left bottom))
   )
+  (text "Put filter Capacitor between L and N. also PPTC fuse and varistor"
+    (at 37.211 37.719 0)
+    (effects (font (size 1.27 1.27) (thickness 0.254) bold) (justify left bottom))
+  )
+  (text "#What's the inductance?" (at 161.544 54.737 0)
+    (effects (font (size 1.27 1.27) (thickness 0.254) bold) (justify left bottom))
+  )
+  (text "Which diode?" (at 162.814 107.823 90)
+    (effects (font (size 1.27 1.27) (thickness 0.254) bold) (justify left bottom))
+  )
+  (text "Which diode?" (at 163.449 70.993 90)
+    (effects (font (size 1.27 1.27) (thickness 0.254) bold) (justify left bottom))
+  )
   (text "POWER SUPPLY\n" (at 101.6 21.59 0)

Commit message: Edited
Parts:
- removed C? (x2): 0.01uF, Capacitor_SMD:C_0603_1608Metric_Pad1.05x0.95mm_HandSolder, symbol Device:C
- removed C? (x2): 0.1uF, Capacitor_SMD:C_0603_1608Metric_Pad1.05x0.95mm_HandSolder, symbol Device:C
- added C1: 0.22uF, Capacitor_THT:C_Rect_L18.0mm_W8.0mm_P15.00mm_FKS3_FKP3, symbol Device:C
- added F1: Fuse, Fuse:Fuse_Bourns_MF-RG300, symbol Device:Fuse
- added RV1: Varistor, Varistor:RV_Disc_D12mm_W4.2mm_P7.5mm, symbol Device:Varistor
- C2, C3: renamed from C?; footprint Capacitor_SMD:CP_Elec_10x10.5 -> Capacitor_SMD:CP_Elec_8x10
- C4, C5: renamed from C?; value 220uF -> 1000uF
- C6, C7: renamed from C?; footprint Capacitor_SMD:C_0603_1608Metric_Pad1.05x0.95mm_HandSolder -> Capacitor_SMD:C_0603_1608Metric
- D2, D3: renamed from D?; value D -> SS34; footprint Diode_SMD:D_SMB -> Diode_SMD:D_SMA
- J1, J2: renamed from J?; footprint MyLibrary:TAB_CONN -> Footprint:TAB_Conn
- L1, L2: renamed from L?; value L -> 47uH; footprint MyLibrary:SRR1208-470YL -> Inductor_SMD:L_12x12mm_H8mm
- R2, R3, R4, R5: renamed from R?; footprint Resistor_SMD:R_0603_1608Metric_Pad1.05x0.95mm_HandSolder -> Resistor_SMD:R_0603_1608Metric
- U1, U2: renamed from U?; footprint Package_TO_SOT_SMD:TO-263-5_TabPin3 -> Package_TO_SOT_SMD:TO-252-5_TabPin3
- gave numbers to parts that had none: 7
Connections:
- net LINE: now also C1.2, F1.2, RV1.1; no longer J2.1 (Pin_1)
- net NEUT: now also C1.1, RV1.2
- new net: F1.1, J2.1 (Pin_1)
Other:
- note removed: "#What's the inductance?"
- note removed: "Put filter Capacitor between L and N. also PPTC fuse and varistor"
- note removed: "Which diode?"
- note removed: "Which one?"
- moved on the sheet: J1, J2, PS1

Commit message: 1
Parts:
- added C10: 15nF, Capacitor_SMD:C_0603_1608Metric, symbol Device:C
- added C8: 100uF, Capacitor_SMD:CP_Elec_8x10, symbol Device:CP
- added C9: 1000uF, Capacitor_SMD:CP_Elec_10x10.5, symbol Device:CP
- added D12: SS34, Diode_SMD:D_SMA, symbol Device:D
- added L3: 47uH, Inductor_SMD:L_12x12mm_H8mm, symbol Device:L
- added R11: 11K, Resistor_SMD:R_0603_1608Metric, symbol Device:R
- added R12: 1.2K, Resistor_SMD:R_0603_1608Metric, symbol Device:R
- added U7: LM2596T-ADJ, Package_TO_SOT_SMD:TO-252-5_TabPin3, symbol Regulator_Switching:LM2596T-ADJ
Connections:
- net +24V: now also R1.2, C8.1, U7.1 (VIN); no longer D1.2 (A)
- net GND: now also D1.1 (K), C8.2, C9.2, D12.2 (A), R12.2, U7.3 (GND), U7.5 (~{ON}/OFF); no longer R1.1
- net LINE: now also F1.1, J2.1 (Pin_1); no longer C1.2, F1.2, PS1.1 (AC/L), RV1.1
- new net: D1.2 (A), R1.1
- new net: D12.1 (K), L3.1, U7.2 (OUT)
- new net: C1.2, F1.2, PS1.1 (AC/L), RV1.1
- new net: C10.1, R11.2, R12.1, U7.4 (FB)
- new net +12V: C10.2, C9.1, L3.2, R11.1
Other:
- note added: "12V"
- moved on the sheet: C2, C25, C26, C3, C4, C5, C6, C7, D1, D2, D3, J2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

Commit message: 1
Parts:
- U1, U2, U7: footprint Package_TO_SOT_SMD:TO-252-5_TabPin3 -> Package_TO_SOT_SMD:TO-263-5_TabPin3
Changed lines of the file:
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@@
     (property "Reference" "U2" (id 0) (at 153.3144 119.3546 0))
     (property "Value" "LM2596T-ADJ" (id 1) (at 153.3144 121.666 0))
-    (property "Footprint" "Package_TO_SOT_SMD:TO-252-5_TabPin3" (id 2) (at 154.5844 135.0264 0)
+    (property "Footprint" "Package_TO_SOT_SMD:TO-263-5_TabPin3" (id 2) (at 154.5844 135.0264 0)
       (effects (font (size 1.27 1.27) italic) (justify left) hide)
     )
@@
     (property "Reference" "U1" (id 0) (at 153.3144 82.5246 0))
     (property "Value" "LM2596T-ADJ" (id 1) (at 153.3144 84.836 0))
-    (property "Footprint" "Package_TO_SOT_SMD:TO-252-5_TabPin3" (id 2) (at 154.5844 98.1964 0)
+    (property "Footprint" "Package_TO_SOT_SMD:TO-263-5_TabPin3" (id 2) (at 154.5844 98.1964 0)
       (effects (font (size 1.27 1.27) italic) (justify left) hide)
     )
@@
     (property "Reference" "U7" (id 0) (at 153.3144 45.212 0))
     (property "Value" "LM2596T-ADJ" (id 1) (at 153.3144 47.5234 0))
-    (property "Footprint" "Package_TO_SOT_SMD:TO-252-5_TabPin3" (id 2) (at 154.5844 60.8838 0)
+    (property "Footprint" "Package_TO_SOT_SMD:TO-263-5_TabPin3" (id 2) (at 154.5844 60.8838 0)
       (effects (font (size 1.27 1.27) italic) (justify left) hide)
     )

Commit message: 1
Connections:
- net +24V: now also D1.2 (A); no longer R1.2
- net GND: now also R1.1; no longer D1.1 (K)
- new net: D1.1 (K), R1.2
Other:
- moved on the sheet: D1, R1
Changed lines of the file:
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@@
     (pin "1")
   )
-  (symbol (lib_id "Device:LED") (at 91.44 49.53 0) (unit 1)
-    (in_bom yes) (on_board yes)
-    (property "Reference" "D1" (id 0) (at 91.44 46.99 0))
-    (property "Value" "LED" (id 1) (at 91.2622 53.6956 0)
-      (effects (font (size 1.27 1.27)) hide)
-    )
-    (property "Footprint" "LED_SMD:LED_0603_1608Metric" (id 2) (at 91.44 49.53 0)
-      (effects (font (size 1.27 1.27)) hide)
-    )
-    (property "Datasheet" "~" (id 3) (at 91.44 49.53 0)
+  (symbol (lib_id "Device:LED") (at 99.06 49.53 0) (unit 1)
+    (in_bom yes) (on_board yes)
+    (property "Reference" "D1" (id 0) (at 99.06 46.99 0))
+    (property "Value" "LED" (id 1) (at 98.8822 53.6956 0)
+      (effects (font (size 1.27 1.27)) hide)
+    )
+    (property "Footprint" "LED_SMD:LED_0603_1608Metric" (id 2) (at 99.06 49.53 0)
+      (effects (font (size 1.27 1.27)) hide)
+    )
+    (property "Datasheet" "~" (id 3) (at 99.06 49.53 0)
       (effects (font (size 1.27 1.27)) hide)
     )
@@
     (pin "4")
   )
-  (symbol (lib_id "Device:R") (at 99.06 49.53 90) (unit 1)
-    (in_bom yes) (on_board yes)
-    (property "Reference" "R1" (id 0) (at 99.06 46.99 90))
-    (property "Value" "4.1K" (id 1) (at 99.1362 49.5554 90))
-    (property "Footprint" "Resistor_SMD:R_0603_1608Metric" (id 2) (at 99.06 51.308 90)
-      (effects (font (size 1.27 1.27)) hide)
-    )
-    (property "Datasheet" "~" (id 3) (at 99.06 49.53 0)
-      (effects (font (size 1.27 1.27)) hide)
-    )
+  (symbol (lib_id "Device:R") (at 91.44 49.53 90) (unit 1)
+    (in_bom yes) (on_board yes)
+    (property "Reference" "R1" (id 0) (at 91.44 46.99 90))
+    (property "Value" "4.1K" (id 1) (at 91.5162 49.5554 90))
+    (property "Footprint" "Resistor_SMD:R_0603_1608Metric" (id 2) (at 91.44 51.308 90)
+      (effects (font (size 1.27 1.27)) hide)
+    )
+    (property "Datasheet" "~" (id 3) (at 91.44 49.53 0)
+      (effects (font (size 1.27 1.27)) hide)
+    )
